File: PCB_Design/Business_Card/Business_Card.kicad_pcb (KiCad board)
At the start: 2 copper layers, 85.6 x 54 mm, 18 parts, among them J1 1-14in IPS ST7789V Display, SW1 Main Power, SW2 SW_Push, SW3 SW_Push, SW4 SW_Push, SW5 SW_Push, U1 XIAO nRF52840

Commit message: PCB Schematic and Layout Updates
Parts:
- J1: footprint Connector_PinHeader_2.54mm:PinHeader_1x08_P2.54mm_Vertical -> GanlathLib:1-14in_IPS_ST7789V_Display
- SW1: footprint Connector_PinHeader_2.54mm:PinHeader_1x02_P2.54mm_Vertical -> GanlathLib:BlankPin_1x02_P2.54mm
- U1: footprint GanlathLib:XIAO-nRF52840-SMD -> GanlathLib:XIAO-nRF52840-SMD_Revised
- moved H4 100.9 mm to (141.0, 75.4)
- moved H3 97.1 mm to (141.0, 30.6)
- moved H2 44.5 mm to (64.6, 75.4)
- moved R2 22.4 mm to (119.7, 48.8), turned to 0 degrees
- moved R1 18.4 mm to (119.7, 51.4), turned to 180 degrees
- moved H1 14.7 mm to (64.6, 30.6)
- moved SW5 12.2 mm to (86.0, 75.5), turned to 180 degrees
- moved R6 12.0 mm to (86.0, 75.5)
- moved SW4 8.66 mm to (101.5, 75.5), turned to 180 degrees
- moved R5 8.51 mm to (101.5, 75.5)
- moved BT1 6.72 mm to (127.7, 31.8)
- moved R4 5.02 mm to (117.0, 75.5)
- moved SW3 5.02 mm to (117.0, 75.5), turned to 180 degrees
- moved SW1 5.01 mm to (134.6, 31.8), turned to 180 degrees
- moved J1 3.16 mm to (88.0, 44.0)
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Connections:
- J1 pad 5: GPIO9 -> GPIO7
- J1 pad 6: GPIO7 -> GPIO9
Routing:
- net GPIO3: track 0.00 -> 67.5 mm, vias 0 -> 1
- net GPIO2: track 0.00 -> 56.6 mm, vias 0 -> 1
- net GPIO9: track 0.00 -> 53.1 mm
- net MOSI: track 0.00 -> 52.2 mm, vias 0 -> 1
- net GPIO7: track 0.00 -> 46.4 mm
- net SCK: track 0.00 -> 45.4 mm, vias 0 -> 1
- net +BATT: track 0.00 -> 44.0 mm
- net GPIO5: track 0.00 -> 43.3 mm
- net GPIO1: track 0.00 -> 43.1 mm, vias 0 -> 1
- net -BATT: track 0.00 -> 39.9 mm
- net GPIO6: track 0.00 -> 39.4 mm
- net GPIO0: track 0.00 -> 32.7 mm, vias 0 -> 1
- net GPIO4: track 0.00 -> 18.7 mm
- net Net-(BT1-Pin_1): track 0.00 -> 6.96 mm
- net +3.3V: track 0.00 -> 3.56 mm, vias 0 -> 1
- added copper zone on F.Cu, net +3.3V
- added copper zone on B.Cu, net GND

Commit message: PCB Revisions
Parts:
- added G***: LOGO, LOGO, F.Cu at (95.7, 54.2)
- added G***: LOGO, LOGO, F.Cu at (136.3, 61.0)
- added G***: LOGO, LOGO, F.Cu at (95.7, 59.6)
- added G*** (x3): LOGO, LOGO, B.Cu at (103.0, 53.5)
- added H5: MountingHole, GanlathLib:MountingHole_3.7mm_Core, F.Cu at (90.0, 30.2)
- added H6: MountingHole, GanlathLib:MountingHole_3.7mm_Lanyard_Core, F.Cu at (102.8, 30.2)
- added H7: MountingHole, GanlathLib:MountingHole_3.7mm_Core, F.Cu at (115.6, 30.2)
- BT1: footprint Connector_JST:JST_XH_B2B-XH-A_1x02_P2.50mm_Vertical -> Connector_PinHeader_2.00mm:PinHeader_2x01_P2.00mm_Vertical_SMD
- H1, H2, H3, H4: footprint MountingHole:MountingHole_3mm -> MountingHole:MountingHole_2.5mm_Pad_TopOnly; moved to B.Cu
- SW1: footprint GanlathLib:BlankPin_1x02_P2.54mm -> Connector_PinHeader_2.00mm:PinHeader_2x01_P2.00mm_Vertical_SMD
- moved SW1 28.6 mm to (113.0, 50.5), turned to 0 degrees
- moved BT1 20.6 mm to (113.0, 46.3), turned to 0 degrees
- moved R2 3.89 mm to (121.0, 45.1), turned to 90 degrees
- moved U1 3.11 mm to (133.7, 45.9)
- moved R1 1.43 mm to (121.0, 50.8), turned to 90 degrees
- moved H1 0.63 mm to (64.2, 30.1)
- moved H2 0.63 mm to (64.2, 75.8)
- moved H3 0.62 mm to (141.4, 30.1)
- moved H4 0.62 mm to (141.4, 75.8)
Routing:
- net +3.3V: track 3.56 -> 173.6 mm, vias 1 -> 4
- net +BATT: track 44.0 -> 30.9 mm
- net -BATT: track 39.9 -> 27.7 mm
- net MOSI: track 52.2 -> 59.9 mm
- net SCK: track 45.4 -> 48.8 mm
- net GPIO0: track 32.7 -> 35.9 mm
- net Net-(BT1-Pin_1): track 6.96 -> 4.24 mm
- net GPIO3: track 67.5 -> 70.2 mm
- net GPIO4: track 18.7 -> 16.3 mm
- net GPIO1: track 43.1 -> 45.4 mm
- net GPIO5: track 43.3 -> 45.1 mm
- net GPIO7: track 46.4 -> 44.8 mm
- net GPIO9: track 53.1 -> 51.8 mm, vias 0 -> 1
- net GPIO6: track 39.4 -> 40.6 mm, vias 0 -> 1
- net GPIO2: track 56.6 -> 57.8 mm
- removed copper zone on F.Cu, net +3.3V
Other:
- board text added: "+"
- board text added: "-"
- board text added: "1-14in IPS ST7789V Display"
- board text added: "B"
- board text added: "Business Card REV: 1.0 Name: Ranil Ganlath S/N:"
- board text added: "C"
- board text added: "D"
- board text added: "DOWN"
- board text added: "G"
- board text added: "LIPO"
- board text added: "M"
- board text added: "MENU"
- board text added: "PWR SW"
- board text added: "R"
- board text added: "Ranil Ganlath"
- board text added: "Robotics | Maker"
- board text added: "S"
- board text added: "SELECT"
- board text added: "Senior Electronics Engineer"
- board text added: "UP"
- board text added: "V"
- board text added: "ranil@ganlath.com"
- board text added: "rganlath3"
